File: Schematics/Working-On/esc v4.1/low_voltage_sch.kicad_sch (KiCad schematic)
At the start: 38 parts, among them IC1 74HCT08BQ,115, IC2 74HCT08BQ,115, U2 ATmega328P-M

Commit message: Ready to order.
Parts:
- added C25: 100n, Capacitor_SMD:C_0402_1005Metric, symbol Device:C
Connections:
- net +5V: now also C16.1, C17.1; no longer C16.2, C17.2
- net GND: now also C16.2, C17.2, C25.1; no longer C16.1, C17.1
- net VBUS: now also C25.2
Other:
- note added: "max_e_speed = 1400 * 60 = 130000 eRPM max_r_speed = 84000 / 7 = 18600 RPM"
- note added: "tan(30) ------------------------------- = 2166 Hz 2 * pi * (33k || 10k + 10k) * 2.4 * 10^(-6)"
- note removed: "max_e_speed = 1400 * 60 = 84000 eRPM max_r_speed = 84000 / 7 = 12000 RPM"
- note removed: "tan(30) --------------------------- = 1400 Hz 2 * pi * (33k || 10k) * 8200 * 10^(-9)"
- moved on the sheet: C16, C17, IC1, IC2, R10, R11, R4, R5, R9
