File: Schematics/Working-On/esc v4.1/esc.kicad_pcb (KiCad board)
At the start: 4 copper layers, 62.5 x 38 mm, 79 parts, among them IC1 74HCT08BQ,115, IC2 74HCT08BQ,115, J1 8730, J10 AVR-ISP-10, J11 Conn_01x06, J2 8730, J3 8730, J4 8730, J5 8730, J6 Conn_01x01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

Commit message: 2 Layers Current Resistor connection.
Routing:
- net Net-(Q6-Pad4): track 29.1 -> 30.1 mm
- net COIL_A_CURR: track 61.6 -> 61.8 mm, vias 2 -> 8
- net COIL_B_CURR: track 37.6 -> 37.8 mm, vias 2 -> 8
- net COIL_C_CURR: vias 4 -> 10
- added copper zone on In2.Cu, net COIL_A_CURR
- added copper zone on In2.Cu, net COIL_B_CURR
- added copper zone on In2.Cu, net COIL_C_CURR
