File: Schematics/Working-On/esc v4.1/high_voltage_sch.kicad_sch (KiCad schematic)
At the start: 21 parts, among them Q1 BSZ0902NS, Q2 BSZ0902NS, Q3 BSZ0902NS, Q4 BSZ0902NS, Q5 BSZ0902NS, Q6 BSZ0902NS, U3 DRV8300DRGER

Commit message: VIA update
Parts:
- R18, R21, R22: value 2m -> 5m
Changed lines of the file:
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@@
 			)
 		)
-		(property "Value" "2m"
+		(property "Value" "5m"
 			(at 192.405 113.03 0)
 			(effects
@@
 			)
 		)
-		(property "Value" "2m"
+		(property "Value" "5m"
 			(at 141.605 113.665 0)
 			(effects
@@
 			)
 		)
-		(property "Value" "2m"
+		(property "Value" "5m"
 			(at 247.015 113.03 0)
 			(effects

Commit message: Ready to order(?)
Parts:
- renumbered C14 to C20, C15 to C21, C16 to C22, C17 to C23, C18 to C24, R12 to R18, R13 to R19, R14 to R20, R15 to R21, R16 to R22, R17 to R23, R21 to R24, R22 to R25, R18 to R26
Changed lines of the file:
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@@
 		(on_board yes)
 		(dnp no)
-		(property "Reference" "C16"
+		(property "Reference" "C22"
 			(at 47.625 73.025 0)
 			(effects
@@
 			(project "esc"
 				(path "/5e78a042-f21c-485f-9078-8bbae1bbdc1b/803d909a-09e2-4af7-89a2-13fdb9464b38"
-					(reference "C16")
+					(reference "C22")
 					(unit 1)
 				)
@@
 		(dnp no)
 		(fields_autoplaced yes)
-		(property "Reference" "R21"
+		(property "Reference" "R24"
 			(at 192.405 110.49 0)
 			(effects
@@
 			(project "esc"
 				(path "/5e78a042-f21c-485f-9078-8bbae1bbdc1b/803d909a-09e2-4af7-89a2-13fdb9464b38"
-					(reference "R21")
+					(reference "R24")
 					(unit 1)
 				)
@@
 		(dnp no)
 		(fields_autoplaced yes)
-		(property "Reference" "#PWR031"
+		(property "Reference" "#PWR048"
 			(at 63.5 67.945 0)
 			(effects
@@
 			(project "esc"
 				(path "/5e78a042-f21c-485f-9078-8bbae1bbdc1b/803d909a-09e2-4af7-89a2-13fdb9464b38"
-					(reference "#PWR031")
+					(reference "#PWR048")
 					(unit 1)
 				)
@@
 		(dnp no)
 		(fields_autoplaced yes)
-		(property "Reference" "#PWR037"
+		(property "Reference" "#PWR054"
 			(at 244.475 123.19 0)
 			(effects
@@
 			(project "esc"
 				(path "/5e78a042-f21c-485f-9078-8bbae1bbdc1b/803d909a-09e2-4af7-89a2-13fdb9464b38"
-					(reference "#PWR037")
+					(reference "#PWR054")
 					(unit 1)
 				)
@@
 		(dnp no)
 		(fields_autoplaced yes)
-		(property "Reference" "C14"
+		(property "Reference" "C20"
 			(at 113.03 61.595 90)
 			(effects
@@
 			(project "esc"
 				(path "/5e78a042-f21c-485f-9078-8bbae1bbdc1b/803d909a-09e2-4af7-89a2-13fdb9464b38"
-					(reference "C14")
+					(reference "C20")
 					(unit 1)
 				)
@@
 		(dnp no)
 		(fields_autoplaced yes)
-		(property "Reference" "#PWR035"
+		(property "Reference" "#PWR051"
 			(at 53.975 85.725 0)
 			(effects
@@
 			(project "esc"
 				(path "/5e78a042-f21c-485f-9078-8bbae1bbdc1b/803d909a-09e2-4af7-89a2-13fdb9464b38"
-					(reference "#PWR035")
+					(reference "#PWR051")
 					(unit 1)
 				)
@@
 		(dnp no)
 		(fields_autoplaced yes)
-		(property "Reference" "#PWR030"
+		(property "Reference" "#PWR047"
 			(at 189.865 58.42 0)
 			(effects
@@
 			(project "esc"
 				(path "/5e78a042-f21c-485f-9078-8bbae1bbdc1b/803d909a-09e2-4af7-89a2-13fdb9464b38"
-					(reference "#PWR030")
+					(reference "#PWR047")
 					(unit 1)
 				)
@@
 		(dnp no)
 		(fields_autoplaced yes)
-		(property "Reference" "#PWR029"
+		(property "Reference" "#PWR046"
 			(at 139.065 45.72 0)
 			(effects
@@
 			(project "esc"
 				(path "/5e78a042-f21c-485f-9078-8bbae1bbdc1b/803d909a-09e2-4af7-89a2-13fdb9464b38"
-					(reference "#PWR029")
+					(reference "#PWR046")
 					(unit 1)
 				)
@@
 		(dnp no)
 		(fields_autoplaced yes)
-		(property "Reference" "#PWR036"
+		(property "Reference" "#PWR053"
 			(at 189.865 123.19 0)
 			(effects
@@
 			(project "esc"
 				(path "/5e78a042-f21c-485f-9078-8bbae1bbdc1b/803d909a-09e2-4af7-89a2-13fdb9464b38"
-					(reference "#PWR036")
+					(reference "#PWR053")
 					(unit 1)
 				)
@@
 		(dnp no)
 		(fields_autoplaced yes)
-		(property "Reference" "R16"
+		(property "Reference" "R22"
 			(at 177.165 83.185 90)
 			(effects
@@
 			(project "esc"
 				(path "/5e78a042-f21c-485f-9078-8bbae1bbdc1b/803d909a-09e2-4af7-89a2-13fdb9464b38"
-					(reference "R16")
+					(reference "R22")
 					(unit 1)
 				)
@@
 		(dnp no)
 		(fields_autoplaced yes)
-		(property "Reference" "R15"
+		(property "Reference" "R21"
 			(at 232.41 72.39 90)
 			(effects
@@
 			(project "esc"
 				(path "/5e78a042-f21c-485f-9078-8bbae1bbdc1b/803d909a-09e2-4af7-89a2-13fdb9464b38"
-					(reference "R15")
+					(reference "R21")
 					(unit 1)
 				)
@@
 		(dnp no)
 		(fields_autoplaced yes)
-		(property "Reference" "#PWR034"
+		(property "Reference" "#PWR050"
 			(at 39.37 85.725 0)
 			(effects
@@
 			(project "esc"
 				(path "/5e78a042-f21c-485f-9078-8bbae1bbdc1b/803d909a-09e2-4af7-89a2-13fdb9464b38"
-					(reference "#PWR034")
+					(reference "#PWR050")
 					(unit 1)
 				)
@@
 		(dnp no)
 		(fields_autoplaced yes)
-		(property "Reference" "R17"
+		(property "Reference" "R23"
 			(at 231.775 95.885 90)
 			(effects
@@
 			(project "esc"
 				(path "/5e78a042-f21c-485f-9078-8bbae1bbdc1b/803d909a-09e2-4af7-89a2-13fdb9464b38"
-					(reference "R17")
+					(reference "R23")
 					(unit 1)
 				)
@@
 		(on_board yes)
 		(dnp no)
-		(property "Reference" "C15"
+		(property "Reference" "C21"
 			(at 35.56 73.025 0)
 			(effects
@@
 			(project "esc"
 				(path "/5e78a042-f21c-485f-9078-8bbae1bbdc1b/803d909a-09e2-4af7-89a2-13fdb9464b38"
-					(reference "C15")
+					(reference "C21")
 					(unit 1)
 				)
@@
 		(dnp no)
 		(fields_autoplaced yes)
-		(property "Reference" "#PWR032"
+		(property "Reference" "#PWR049"
 			(at 244.475 71.12 0)
 			(effects
@@
 			(project "esc"
 				(path "/5e78a042-f21c-485f-9078-8bbae1bbdc1b/803d909a-09e2-4af7-89a2-13fdb9464b38"
-					(reference "#PWR032")
+					(reference "#PWR049")
 					(unit 1)
 				)
@@
 		(dnp no)
 		(fields_autoplaced yes)
-		(property "Reference" "#PWR040"
+		(property "Reference" "#PWR052"
 			(at 107.95 120.015 0)
 			(effects
@@
 			(project "esc"
 				(path "/5e78a042-f21c-485f-9078-8bbae1bbdc1b/803d909a-09e2-4af7-89a2-13fdb9464b38"
-					(reference "#PWR040")
+					(reference "#PWR052")
 					(unit 1)
 				)
@@
 		(dnp no)
 		(fields_autoplaced yes)
-		(property "Reference" "R18"
+		(property "Reference" "R26"
 			(at 141.605 111.125 0)
 			(effects
@@
 			(project "esc"
 				(path "/5e78a042-f21c-485f-9078-8bbae1bbdc1b/803d909a-09e2-4af7-89a2-13fdb9464b38"
-					(reference "R18")
+					(reference "R26")
 					(unit 1)
 				)
@@
 		(dnp no)
 		(fields_autoplaced yes)
-		(property "Reference" "C17"
+		(property "Reference" "C23"
 			(at 163.83 74.295 90)
 			(effects
@@
 			(project "esc"
 				(path "/5e78a042-f21c-485f-9078-8bbae1bbdc1b/803d909a-09e2-4af7-89a2-13fdb9464b38"
-					(reference "C17")
+					(reference "C23")
 					(unit 1)
 				)
@@
 		(dnp no)
 		(fields_autoplaced yes)
-		(property "Reference" "R14"
+		(property "Reference" "R20"
 			(at 126.365 70.485 90)
 			(effects
@@
 			(project "esc"
 				(path "/5e78a042-f21c-485f-9078-8bbae1bbdc1b/803d909a-09e2-4af7-89a2-13fdb9464b38"
-					(reference "R14")
+					(reference "R20")
 					(unit 1)
 				)
@@
 		(dnp no)
 		(fields_autoplaced yes)
-		(property "Reference" "#PWR033"
+		(property "Reference" "#PWR055"
 			(at 139.065 123.825 0)
 			(effects
@@
 			(project "esc"
 				(path "/5e78a042-f21c-485f-9078-8bbae1bbdc1b/803d909a-09e2-4af7-89a2-13fdb9464b38"
-					(reference "#PWR033")
+					(reference "#PWR055")
 					(unit 1)
 				)
@@
 		(dnp no)
 		(fields_autoplaced yes)
-		(property "Reference" "R12"
+		(property "Reference" "R18"
 			(at 127 46.609 90)
 			(effects
@@
 			(project "esc"
 				(path "/5e78a042-f21c-485f-9078-8bbae1bbdc1b/803d909a-09e2-4af7-89a2-13fdb9464b38"
-					(reference "R12")
+					(reference "R18")
 					(unit 1)
 				)
@@
 		(dnp no)
 		(fields_autoplaced yes)
-		(property "Reference" "R22"
+		(property "Reference" "R25"
 			(at 247.015 110.49 0)
 			(effects
@@
 			(project "esc"
 				(path "/5e78a042-f21c-485f-9078-8bbae1bbdc1b/803d909a-09e2-4af7-89a2-13fdb9464b38"
-					(reference "R22")
+					(reference "R25")
 					(unit 1)
 				)
@@
 		(dnp no)
 		(fields_autoplaced yes)
-		(property "Reference" "R13"
+		(property "Reference" "R19"
 			(at 177.8 59.69 90)
 			(effects
@@
 			(project "esc"
 				(path "/5e78a042-f21c-485f-9078-8bbae1bbdc1b/803d909a-09e2-4af7-89a2-13fdb9464b38"
-					(reference "R13")
+					(reference "R19")
 					(unit 1)
 				)
@@
 		(dnp no)
 		(fields_autoplaced yes)
-		(property "Reference" "C18"
+		(property "Reference" "C24"
 			(at 218.44 86.995 90)
 			(effects
@@
 			(project "esc"
 				(path "/5e78a042-f21c-485f-9078-8bbae1bbdc1b/803d909a-09e2-4af7-89a2-13fdb9464b38"
-					(reference "C18")
-					(unit 1)
-				)
+					(reference "C24")
+					(unit 1)
+				)

Commit message: Changing the VD Resistors to 3.33k.
Parts:
- R24, R25, R26: value 5m -> 20m
Changed lines of the file:
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@@
 			)
 		)
-		(property "Value" "5m"
+		(property "Value" "20m"
 			(at 192.405 113.03 0)
 			(effects
@@
 			)
 		)
-		(property "Value" "5m"
+		(property "Value" "20m"
 			(at 141.605 113.665 0)
 			(effects
@@
 			)
 		)
-		(property "Value" "5m"
+		(property "Value" "20m"
 			(at 247.015 113.03 0)
 			(effects
