File: Schematics/filters.kicad_sch (KiCad schematic)
At the start: 20 parts

Commit message: Cleaning up.
Other:
- note added: "max_e_speed = 1860 * 60 = 111600 eRPM max_r_speed = 111600 / 7 = 15940 RPM"
- note added: "tan(30) ------------------------------- = 1860 Hz 2 * pi * (33k || 20k + 10k) * 2.2 * 10^(-6)"
- note removed: "max_e_speed = 2363 * 60 = 141720 eRPM max_r_speed = 84000 / 7 = 20245 RPM"
- note removed: "tan(30) ------------------------------- = 2363 Hz 2 * pi * (33k || 10k + 10k) * 2.2 * 10^(-6)"
Changed lines of the file:
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@@
 		)
 	)
-	(text "tan(30)\n            ------------------------------- = 2363 Hz\n2 * pi * (33k || 10k + 10k) * 2.2 * 10^(-6)"
+	(text "tan(30)\n            ------------------------------- = 1860 Hz\n2 * pi * (33k || 20k + 10k) * 2.2 * 10^(-6)"
 		(exclude_from_sim no)
 		(at 99.314 44.196 0)
@@
 		)
 	)
-	(text "max_e_speed = 2363 * 60 = 141720 eRPM\nmax_r_speed = 84000 / 7 =  20245 RPM  "
+	(text "max_e_speed = 1860 * 60  = 111600 eRPM\nmax_r_speed = 111600 / 7 =  15940 RPM  "
 		(exclude_from_sim no)
 		(at 75.692 49.784 0)
