File: Schematics/Pages/filters.kicad_sch (KiCad schematic)
At the start: 20 parts

Commit message: V1.0
Parts:
- renumbered R2 to R1, R4 to R12, R7 to R14, R1 to R15, R8 to R2, R5 to R3, R14 to R4, R15 to R5, R3 to R6, R12 to R7, R6 to R8
Connections:
- net COIL_A: now also R2.1; no longer R2.2
- net COIL_A_BEMF: now also R1.1; no longer R1.2
- net COIL_B: now also R7.1; no longer R7.2
- net COIL_B_BEMF: now also R6.1; no longer R6.2
- net COIL_C: now also R13.1; no longer R13.2
- net COIL_C_BEMF: now also R12.1; no longer R12.2
- new net: R1.2, R2.2, R3.2
- new net: R6.2, R7.2, R8.2
- new net: R12.2, R13.2, R14.2
Other:
- moved on the sheet: C13, C14, C15, R13, R14, R2, R3, R7, R8
