File: Schematics/Pages/high_voltage_sch.kicad_sch (KiCad schematic)
At the start: 21 parts, among them Q1 BSZ0902NS, Q2 BSZ0902NS, Q3 BSZ0902NS, Q4 BSZ0902NS, Q5 BSZ0902NS, Q6 BSZ0902NS, U3 DRV8300DRGER

Commit message: V1.0
Parts:
- C20, C23, C24: value 4700p -> 0.1u
- R24, R25, R26: value 20m -> 5m
- renumbered Q1 to AH1, Q3 to AL1, Q2 to BH1, Q5 to BL1, Q4 to CH1, Q6 to CL1
Changed lines of the file:
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@@
 		(dnp no)
 		(fields_autoplaced yes)
-		(property "Reference" "Q5"
+		(property "Reference" "BL1"
 			(at 192.786 78.74 0)
 			(effects
@@
 			(project "esc"
 				(path "/5e78a042-f21c-485f-9078-8bbae1bbdc1b/803d909a-09e2-4af7-89a2-13fdb9464b38"
-					(reference "Q5")
+					(reference "BL1")
 					(unit 1)
 				)
@@
 			)
 		)
-		(property "Value" "20m"
+		(property "Value" "5m"
 			(at 192.405 113.03 0)
 			(effects
@@
 			)
 		)
-		(property "Value" "4700p"
+		(property "Value" "0.1u"
 			(at 113.03 64.135 90)
 			(effects
@@
 		(dnp no)
 		(fields_autoplaced yes)
-		(property "Reference" "Q4"
+		(property "Reference" "CH1"
 			(at 248.285 74.93 0)
 			(effects
@@
 			(project "esc"
 				(path "/5e78a042-f21c-485f-9078-8bbae1bbdc1b/803d909a-09e2-4af7-89a2-13fdb9464b38"
-					(reference "Q4")
+					(reference "CH1")
 					(unit 1)
 				)
@@
 		(dnp no)
 		(fields_autoplaced yes)
-		(property "Reference" "Q6"
+		(property "Reference" "CL1"
 			(at 247.396 91.44 0)
 			(effects
@@
 			(project "esc"
 				(path "/5e78a042-f21c-485f-9078-8bbae1bbdc1b/803d909a-09e2-4af7-89a2-13fdb9464b38"
-					(reference "Q6")
+					(reference "CL1")
 					(unit 1)
 				)
@@
 		(dnp no)
 		(fields_autoplaced yes)
-		(property "Reference" "Q1"
+		(property "Reference" "AH1"
 			(at 142.24 49.1489 0)
 			(effects
@@
 			(project "esc"
 				(path "/5e78a042-f21c-485f-9078-8bbae1bbdc1b/803d909a-09e2-4af7-89a2-13fdb9464b38"
-					(reference "Q1")
+					(reference "AH1")
 					(unit 1)
 				)
@@
 		(dnp no)
 		(fields_autoplaced yes)
-		(property "Reference" "Q2"
+		(property "Reference" "BH1"
 			(at 192.786 62.23 0)
 			(effects
@@
 			(project "esc"
 				(path "/5e78a042-f21c-485f-9078-8bbae1bbdc1b/803d909a-09e2-4af7-89a2-13fdb9464b38"
-					(reference "Q2")
+					(reference "BH1")
 					(unit 1)
 				)
@@
 			)
 		)
-		(property "Value" "20m"
+		(property "Value" "5m"
 			(at 141.605 113.665 0)
 			(effects
@@
 			)
 		)
-		(property "Value" "4700p"
+		(property "Value" "0.1u"
 			(at 163.83 76.835 90)
 			(effects
@@
 			)
 		)
-		(property "Value" "20m"
+		(property "Value" "5m"
 			(at 247.015 113.03 0)
 			(effects
@@
 			)
 		)
-		(property "Value" "4700p"
+		(property "Value" "0.1u"
 			(at 218.44 89.535 90)
 			(effects
@@
 		(dnp no)
 		(fields_autoplaced yes)
-		(property "Reference" "Q3"
+		(property "Reference" "AL1"
 			(at 142.875 65.405 0)
 			(effects
@@
 			(project "esc"
 				(path "/5e78a042-f21c-485f-9078-8bbae1bbdc1b/803d909a-09e2-4af7-89a2-13fdb9464b38"
-					(reference "Q3")
-					(unit 1)
-				)
+					(reference "AL1")
+					(unit 1)
+				)
