File: Schematics/Pages/low_voltage_sch.kicad_sch (KiCad schematic)
At the start: 19 parts, among them IC1 74HCT08BQ,115, IC2 74HCT08BQ,115, U2 ATmega328P-M

Commit message: V1.0
Parts:
- renumbered C17 to C16, C16 to C17, R16 to R27, R17 to R28, 8MHz1 to XTAL1
Changed lines of the file:
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@@
 		(on_board yes)
 		(dnp no)
-		(property "Reference" "C16"
+		(property "Reference" "C17"
 			(at 64.516 49.784 0)
 			(effects
@@
 			(project "esc"
 				(path "/5e78a042-f21c-485f-9078-8bbae1bbdc1b/9f25a095-da1c-4b42-a0b8-dca0a87bd952"
-					(reference "C16")
+					(reference "C17")
 					(unit 1)
 				)
@@
 		(on_board yes)
 		(dnp no)
-		(property "Reference" "C17"
+		(property "Reference" "C16"
 			(at 64.6938 103.9368 0)
 			(effects
@@
 			(project "esc"
 				(path "/5e78a042-f21c-485f-9078-8bbae1bbdc1b/9f25a095-da1c-4b42-a0b8-dca0a87bd952"
-					(reference "C17")
+					(reference "C16")
 					(unit 1)
 				)
@@
 		(on_board yes)
 		(dnp no)
-		(property "Reference" "R17"
+		(property "Reference" "R28"
 			(at 229.87 128.397 90)
 			(effects
@@
 			(project "esc"
 				(path "/5e78a042-f21c-485f-9078-8bbae1bbdc1b/9f25a095-da1c-4b42-a0b8-dca0a87bd952"
-					(reference "R17")
+					(reference "R28")
 					(unit 1)
 				)
@@
 		(on_board yes)
 		(dnp no)
-		(property "Reference" "R16"
+		(property "Reference" "R27"
 			(at 238.76 113.03 90)
 			(effects
@@
 			(project "esc"
 				(path "/5e78a042-f21c-485f-9078-8bbae1bbdc1b/9f25a095-da1c-4b42-a0b8-dca0a87bd952"
-					(reference "R16")
+					(reference "R27")
 					(unit 1)
 				)
@@
 		(dnp no)
 		(fields_autoplaced yes)
-		(property "Reference" "8MHz1"
+		(property "Reference" "XTAL1"
 			(at 193.675 40.64 0)
 			(effects
@@
 			(project "esc"
 				(path "/5e78a042-f21c-485f-9078-8bbae1bbdc1b/9f25a095-da1c-4b42-a0b8-dca0a87bd952"
-					(reference "8MHz1")
-					(unit 1)
-				)
+					(reference "XTAL1")
+					(unit 1)
+				)
